File: Hardware/Master_Clock/Master_Clock.kicad_sch (KiCad schematic)
At the start: 9 parts, among them U1 LT8330

Commit message: Finished Schematic.
Parts:
- added C10, C11, C12, C7, C8, C9: 100nF 50V, symbol Device:C
- added C13: 4.7pF 50V, symbol Device:C
- added C14: 470u 50V, Capacitor_THT:C_Radial_D12.5mm_H25.0mm_P5.00mm, symbol Device:C_Polarized
- added C5, C6: 4u7 X5R 50V, Capacitor_SMD:C_0805_2012Metric_Pad1.18x1.45mm_HandSolder, symbol Device:C
- added D1: LG L29K, LED_SMD:LED_0603_1608Metric_Pad1.05x0.95mm_HandSolder, symbol Device:LED
- added J1: Conn_01x03_Pin, Connector_PinHeader_2.54mm:PinHeader_1x03_P2.54mm_Vertical, symbol Connector:Conn_01x03_Pin
- added J2, J3: Screw_Terminal_01x02, symbol Connector:Screw_Terminal_01x02
- added Q1: BC847, Package_TO_SOT_SMD:SOT-23, symbol Transistor_BJT:BC847
- added R10, R9: 10M 1%, Resistor_SMD:R_0603_1608Metric_Pad0.98x0.95mm_HandSolder, symbol Device:R
- added R3, R4, R5: 10k, Resistor_SMD:R_0603_1608Metric_Pad0.98x0.95mm_HandSolder, symbol Device:R
- added R6, R8: 2k2, Resistor_SMD:R_0603_1608Metric_Pad0.98x0.95mm_HandSolder, symbol Device:R
- added R7: 470R, Resistor_SMD:R_0603_1608Metric_Pad0.98x0.95mm_HandSolder, symbol Device:R
- added SW1, SW2: SW_Push, Button_Switch_THT:SW_PUSH_6mm, symbol Switch:SW_Push
- added TP1: 32kHz, symbol Connector:TestPoint
- added TP2: MinPulse, symbol Connector:TestPoint
- added U2: ATtiny402-SS, Package_SO:SOIC-8_3.9x4.9mm_P1.27mm, symbol MCU_Microchip_ATtiny:ATtiny402-SS
- added U3: AP7370-18W5, Package_TO_SOT_SMD:SOT-23-5, symbol Master_Clock:AP7370-18W5
- added U4: LT1178S8, Package_SO:SOIC-8_3.9x4.9mm_P1.27mm, symbol Master_Clock:LT1178S8
- added U5: OP193, Package_SO:SOIC-8_3.9x4.9mm_P1.27mm, symbol Master_Clock:OP193
- added X1: SG-3031CM, Oscillator:Oscillator_SMD_SeikoEpson_SG3030CM, symbol Oscillator:SG-3030CM
- R1: value 1M 1% -> 10M 1%
- R2: value 75k 1% -> 750k 1%
Connections:
- net GND: now also C10.2, C11.2, C12.2, C5.2, C6.2, C7.2, C8.2, C9.2, J1.3 (Pin_3), J2.2 (Pin_2), J3.2 (Pin_2), Q1.2 (E), R10.2, R8.2, SW1.2, SW2.2, U2.8 (GND), U3.2 (GND), U4.2 (V-), U4.4 (-), U5.4 (V-), X1.2 (GND)
- net at R1.2, R2.1, U1.3 (FBX): now also C13.2
- net +24V: now reaches C2.1, C4.1, D2.1 (K), R1.1
- net +24V: now also C13.1, U4.6 (V+), U5.7 (V+)
- net +BATT: now reaches C1.1, L1.1, U1.4 (EN/UVLO), U1.6 (Vin)
- net +BATT: now also C5.1, J2.1 (Pin_1), R6.1, U3.1 (VI)
- new net: D1.2 (A), R6.2
- new net: C11.1, R4.2, SW2.1, U2.3 (PA7)
- new net: C12.1, R5.2, SW1.1, U2.2 (PA6)
- new net: R7.1, U2.5 (PA2)
- new net: TP1.1, U2.7 (PA3), X1.3 (OUT)
- new net: C14.2, J3.1 (Pin_1)
- new net: C14.1, U4.7, U5.6
- new net: R10.1, R9.2, U4.8 (-), U5.2 (-)
- new net: Q1.1 (B), R7.2, R8.1
- new net: D1.1 (K), Q1.3 (C)
- new net +1V8: C6.1, C7.1, C8.1, C9.1, J1.1 (Pin_1), R3.1, R4.1, R5.1, R9.1, U2.1 (VCC), U3.5 (VO), U4.3 (+), X1.1 (VIO), X1.4 (Vcc)
- new net WO1: TP2.1, U2.4 (PA1), U4.1 (+), U5.3 (+)
- new net ~{RESET}/UPDI: C10.1, J1.2 (Pin_2), R3.2, U2.6 (~{RESET}/PA0)
- no-connect marks 0 -> 2
Other:
- note added: "3 ... 10 V"
- note added: "Alternative: ASH7KW-32.768KHZ-L-T"
- note added: "Slave Clock"
- note added: "UPDI"
- note removed: "3 ... 12V"
- company: (none) -> Christian Mauderer
- title: (none) -> Master Clock
- moved on the sheet: C1, C2, C3, C4, D2, L1, R1, R2, U1

Commit message: BOM and DigiKey numbers.
Parts:
- added TP1: OPOut, TestPoint:TestPoint_Pad_D1.0mm, symbol Connector:TestPoint
- C1: renamed from C13; footprint (none) -> Capacitor_SMD:C_0603_1608Metric_Pad1.08x0.95mm_HandSolder
- C10, C11, C12, C7: footprint (none) -> Capacitor_SMD:C_0603_1608Metric_Pad1.08x0.95mm_HandSolder
- C13: renamed from C9; footprint (none) -> Capacitor_SMD:C_0603_1608Metric_Pad1.08x0.95mm_HandSolder
- C14: renamed from C8; footprint (none) -> Capacitor_SMD:C_0603_1608Metric_Pad1.08x0.95mm_HandSolder
- J1: renamed from J2; value Screw_Terminal_01x02 -> Phoenix Contact 1935161; footprint (none) -> TerminalBlock_Phoenix:TerminalBlock_Phoenix_PT-1,5-2-5.0-H_1x02_P5.00mm_Horizontal
- J2: renamed from J3; value Screw_Terminal_01x02 -> Phoenix Contact 1935161; footprint (none) -> TerminalBlock_Phoenix:TerminalBlock_Phoenix_PT-1,5-2-5.0-H_1x02_P5.00mm_Horizontal
- TP2: footprint (none) -> TestPoint:TestPoint_Pad_D1.0mm
- TP3: renamed from TP1; footprint (none) -> TestPoint:TestPoint_Pad_D1.0mm
- U3: renamed from U5; value OP193 -> OP193FS
- renumbered C1 to C2, C2 to C3, C14 to C5, C3 to C6, C5 to C8, C6 to C9, D2 to D1, D1 to D2, J1 to J3, R9 to R1, R8 to R10, R1 to R2, R10 to R3, R2 to R4, R6 to R5, R3 to R6, R4 to R7, R5 to R8, R7 to R9, SW2 to SW1, SW1 to SW2, U4 to U1, U1 to U2, U3 to U4, U2 to U5
Connections:
- net Key2: now reaches C11.1, R7.2, SW1.1, U5.3 (PA7)
- net Key1: now reaches C12.1, R8.2, SW2.1, U5.2 (PA6)
- net LED: now reaches R9.1, U5.5 (PA2)
- net 32kHz: now reaches TP3.1, U5.7 (PA3), X1.3 (OUT)
- net SlaveClock: now reaches C5.2, J2.1 (Pin_1)
- net at C5.1, U1.7, U3.6: now also TP1.1
- net WO1 renamed MinPulse
- no-connect marks 2 -> 3

Commit message: HW V1.0.
Parts:
- removed TP1: OPOut, TestPoint:TestPoint_Pad_D1.0mm, symbol Connector:TestPoint
- added H1, H2: MountingHole, MountingHole:MountingHole_3.2mm_M3_ISO7380_Pad, symbol Mechanical:MountingHole
- added R11, R12: 0R, Resistor_SMD:R_0603_1608Metric_Pad0.98x0.95mm_HandSolder, symbol Device:R
- renumbered TP3 to TP1
Connections:
- net +BATT: now also D2.2 (A), R12.2; no longer R5.1, U2.4 (EN/UVLO)
- net Key1: now also C11.1, R7.2, SW1.1; no longer C12.1, R8.2, SW2.1
- net Key2: now also C12.1, R8.2, SW2.1; no longer C11.1, R7.2, SW1.1
- net at R5.2: now also Q1.3 (C); no longer D2.2 (A)
- net at U1.7, U3.6: now also R11.1; no longer C5.1
- net at D2.1 (K): now also R5.1; no longer Q1.3 (C)
- new net: C5.1, R11.2
- new net: R12.1, U2.4 (EN/UVLO)
Other:
- note added: "PAUSE"
- note added: "STEP"
- moved on the sheet: C5, D2, R5

Commit message: HW V1.0-2023-12-28 - Add 0R-resistors in supply.
Parts:
- added R13, R14: 0R, Resistor_SMD:R_0603_1608Metric_Pad0.98x0.95mm_HandSolder, symbol Device:R
Connections:
- net +BATT: now also R13.2, R14.2; no longer C2.1, C8.1, L1.1, R12.2, U2.6 (Vin), U4.1 (VI)
- new net: C8.1, R14.1, U4.1 (VI)
- new net: C2.1, L1.1, R12.2, R13.1, U2.6 (Vin)
Other:
- moved on the sheet: C1, C2, C3, C4, C5, C6, D1, J1, J2, L1, R1, R11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

Commit message: Hardware 1.1
Parts:
- added R15, R16, R17: 2M2, Resistor_SMD:R_0603_1608Metric_Pad0.98x0.95mm_HandSolder, symbol Device:R
- C4: now not fitted
- C5: value 470u 50V -> Panasonic FC 180u 63V
- R1, R3: value 10M 1% -> 2M2
- R2: value 10M 1% -> 4M7
- R4: value 750k 1% -> 330k
Connections:
- net +1V8: now also R16.1
- net GND: now also R17.2
- net MinPulse: now also R15.1; no longer U1.1 (+), U3.3 (+)
- new net: R15.2, R16.2, R17.1, U1.1 (+), U3.3 (+)
Other:
- note added: "4M7 / 330k -> 24.4V 2M2 / 330k -> 12.3V"
- note removed: "1M / 75k -> 23V 1M / 150k -> 12.3V"
- moved on the sheet: C1, C2, C3, C6, D1, J1, L1, R1, R12, R13, R2, R3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
